File: KiCAD/Altoids.kicad_pcb (KiCad board)
At the start: 2 copper layers, 91.4 x 50.8 mm, 55 parts, among them J1 Conn_01x04_Pin, J10 Conn_01x01, J11 Conn_01x01, J12 Conn_01x01, J13 Conn_01x01, J14 Conn_01x02, J15 Conn_01x02, J16 Conn_01x04_Pin, J17 Conn_01x10_Pin, J18 Conn_01x02, J19 Conn_01x03_Pin, J2 UART, J20 1802, J21 Power, J22 UART, J23 CLK, J24 Conn_01x05, J3 UART, J4 Conn_01x01, J5 Conn_01x01, J6 Conn_01x01, J7 Conn_01x01, J8 Conn_01x01, J9 Conn_01x01, SW1 BAT, SW2 VCC, SW3 UART, SW4 LOGIC, SW5 CLK, SW6 SIGNAL, U1 FT232RL, U2 PIC12F629

Commit message: WIP
Parts:
- removed J10, J11, J12, J13, J5, J6, J7, J8, J9: Conn_01x01, TestPoint:TestPoint_THTPad_D1.5mm_Drill0.7mm_SLOTTED
- J1: value Conn_01x04_Pin -> 3V3 Reg
- J16: value Conn_01x04_Pin -> 5V Reg
- J17: value Conn_01x10_Pin -> Power Mux
- J4: value Conn_01x01 -> Lipo Amigo Pro; footprint TestPoint:TestPoint_THTPad_D1.5mm_Drill0.7mm_SLOTTED -> Connector_PinHeader_2.54mm:PinHeader_1x10_P2.54mm_Vertical
- moved J4 0.10 mm to (102.5, 81.6), turned to 90 degrees
