File: KiCAD/Altoids.kicad_sch (KiCad schematic)
At the start: 53 parts, among them J1 Conn_01x04_Pin, J10 Conn_01x01, J11 Conn_01x01, J12 Conn_01x01, J13 Conn_01x01, J14 Conn_01x02, J15 Conn_01x02, J16 Conn_01x04_Pin, J17 Conn_01x10_Pin, J18 Conn_01x02, J19 Conn_01x03_Pin, J2 UART, J20 1802, J21 Power, J22 UART, J23 CLK, J24 Conn_01x05, J3 UART, J4 Conn_01x01, J5 Conn_01x01, J6 Conn_01x01, J7 Conn_01x01, J8 Conn_01x01, J9 Conn_01x01, SW1 BAT, SW2 VCC, SW3 UART, SW4 LOGIC, SW5 CLK, SW6 SIGNAL, U1 FT232RL, U2 PIC12F629

Commit message: WIP
Parts:
- removed J10, J11, J12, J13, J4, J5, J6, J7, J8, J9: Conn_01x01, TestPoint:TestPoint_THTPad_D1.5mm_Drill0.7mm_SLOTTED, symbol Connector_Generic:Conn_01x01
- added J4: Lipo Amigo Pro, Connector_PinHeader_2.54mm:PinHeader_1x10_P2.54mm_Vertical, symbol Connector_Generic:Conn_01x10
- J1: value Conn_01x04_Pin -> 3V3 Reg
- J16: value Conn_01x04_Pin -> 5V Reg
- J17: value Conn_01x10_Pin -> Power Mux
Connections:
- net CHG: now also J4.3 (Pin_3)
- net GND: now also J4.1 (Pin_1), J4.5 (Pin_5), J4.8 (Pin_8)
- net ON: now also J4.4 (Pin_4)
- net SW_POWER_A: now also J4.9 (Pin_9)
- net SW_POWER_B: now also J4.10 (Pin_10)
- net VBAT: now also J4.7 (Pin_7)
- net VBUS: now also J4.2 (Pin_2)
- net VDEV: now also J4.6 (Pin_6)
Other:
- company: (none) -> by AdamT117 https://github.com/Kayto
- title: (none) -> Altoids Serial Adaper SCHEMATIC
