File: KiCAD/Altoids_TOP.kicad_pcb (KiCad board)
At the start: 2 copper layers, 91.4 x 50.8 mm, 0 parts

Commit message: WIP
Other:
- outline, holes or cut-outs redrawn
- board text added: "0V"
- board text added: "600 hZ"
- board text added: "6MhZ"
- board text added: "DAT"
- board text added: "PIC PROG"
- board text added: "Vdd"
- board text added: "Vpp"
- board text added: "bLah"
